File: 2SteppersESP32.kicad_pcb (KiCad board)
At the start: 2 copper layers, 69 x 58.5 mm, 50 parts, among them J1 LED_Strip, J10 I2C, J2 Dallas, J3 I2C, J4 INPUT, J5 POWER_IN, J6 MOTOR, J7 MOTOR, J8 OUT_IO, J9 INPUT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

Commit message: pcb upate
Other:
- board text added: "28V Max!"
- board text added: "Digi IO"
- board text added: "Set to 5v BEFORE inserting."
Changed lines of the file:
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@@
 		)
 	)
-	(gr_text "Dallas"
-		(at 146.92 83.7 -90)
+	(gr_text "Digi IO"
+		(at 146.92 83.7 270)
 		(layer "F.SilkS")
 		(effects
@@
 		)
 	)
+	(gr_text "28V Max!"
+		(at 204.5 100 90)
+		(layer "F.Mask")
+		(effects
+			(font
+				(size 1 1)
+				(thickness 0.15)
+			)
+			(justify left bottom)
+		)
+	)
+	(gr_text "Set to 5v\nBEFORE inserting."
+		(at 170 98.5 90)
+		(layer "F.Mask")
+		(effects
+			(font
+				(size 1 1)
+				(thickness 0.15)
+			)
+			(justify left bottom)
+		)
+	)
